Commit message: updated my self design of an ackermann robot using openscad and ROS2 Jazzy and Gazebo Harmonic and Jetty

File: model.urdf (robot description, URDF)
Before this commit: robot ackermann_robot, 8 links, 7 joints
Links:
- link chassis_link: mass 0.126 -> 0.13442; geometry collision box size=0.27 0.1205 0.01; visual cylinder length=0.04 radius=0.004
- link front_left_wheel_link: mass 0.05 -> 0.0677; geometry collision cylinder length=0.03 radius=0.036; visual mesh filename=/home/mohana/robot_ws/src/ackermann_robot/meshes/front_left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 scale=0.001 0.001 0.001
- link front_right_wheel_link: mass 0.05 -> 0.0677; geometry collision cylinder length=0.03 radius=0.036; visual mesh filename=/home/mohana/robot_ws/src/ackermann_robot/meshes/front_righ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 scale=0.001 0.001 0.001
- link rear_left_wheel_link: mass 0.05 -> 0.0677; geometry collision cylinder length=0.03 radius=0.036; visual mesh filename=/home/mohana/robot_ws/src/ackermann_robot/meshes/rear_left_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 scale=0.001 0.001 0.001
- link rear_right_wheel_link: mass 0.05 -> 0.0677; geometry collision cylinder length=0.03 radius=0.036; visual mesh filename=/home/mohana/robot_ws/src/ackermann_robot/meshes/rear_right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 scale=0.001 0.001 0.001
Joints:
- joint base_to_chassis: origin xyz=0 0 0.0375 rpy=0 0 0 -> xyz=0 0 0.036 rpy=0 0 0
- joint front_left_steer_joint: limit lower=-0.6 upper=0.6 effort=25 velocity=2 -> (none); origin xyz=0.095 0.076 0.0375 -> xyz=0.1025 0.076 0.036
- joint front_left_wheel_joint: limit effort=10 velocity=10 -> (none); type revolute -> continuous
- joint front_right_steer_joint: limit lower=-0.6 upper=0.6 effort=25 velocity=2 -> (none); origin xyz=0.095 -0.076 0.0375 -> xyz=0.1025 -0.076 0.036
- joint front_right_wheel_joint: limit effort=10 velocity=10 -> (none); type revolute -> continuous
- joint rear_left_wheel_joint: limit effort=10 velocity=10 -> (none); origin xyz=-0.095 0.076 0.0375 -> xyz=-0.1025 0.076 0.036; type revolute -> continuous
- joint rear_right_wheel_joint: limit effort=10 velocity=10 -> (none); origin xyz=-0.095 -0.076 0.0375 -> xyz=-0.1025 -0.076 0.036; type revolute -> continuous

File: src/ackermann_robot/urdf/ackermann_robot.urdf (robot description, URDF)
Before this commit: robot ackermann_robot, 8 links, 7 joints
Links:
- link chassis_link: mass 0.126 -> 0.13442; geometry collision box size=0.27 0.1205 0.01; visual cylinder length=0.04 radius=0.004
- link front_left_wheel_link: mass 0.05 -> 0.0677; geometry collision cylinder length=0.03 radius=0.036; visual mesh filename=/home/mohana/robot_ws/src/ackermann_robot/meshes/front_left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 scale=0.001 0.001 0.001
- link front_right_wheel_link: mass 0.05 -> 0.0677; geometry collision cylinder length=0.03 radius=0.036; visual mesh filename=/home/mohana/robot_ws/src/ackermann_robot/meshes/front_righ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 scale=0.001 0.001 0.001
- link rear_left_wheel_link: mass 0.05 -> 0.0677; geometry collision cylinder length=0.03 radius=0.036; visual mesh filename=/home/mohana/robot_ws/src/ackermann_robot/meshes/rear_left_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 scale=0.001 0.001 0.001
- link rear_right_wheel_link: mass 0.05 -> 0.0677; geometry collision cylinder length=0.03 radius=0.036; visual mesh filename=/home/mohana/robot_ws/src/ackermann_robot/meshes/rear_right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 scale=0.001 0.001 0.001
Joints:
- joint base_to_chassis: origin xyz=0 0 0.0375 rpy=0 0 0 -> xyz=0 0 0.036 rpy=0 0 0
- joint front_left_steer_joint: limit lower=-0.6 upper=0.6 effort=25 velocity=2 -> lower=-0.6 upper=0.6 effort=1 velocity=2; origin xyz=0.095 0.076 0.0375 -> xyz=0.1025 0.076 0.036
- joint front_left_wheel_joint: limit effort=10 velocity=10 -> lower=-1.5708 upper=1.5708 effort=1 velocity=10
- joint front_right_steer_joint: limit lower=-0.6 upper=0.6 effort=25 velocity=2 -> lower=-0.6 upper=0.6 effort=1 velocity=2; origin xyz=0.095 -0.076 0.0375 -> xyz=0.1025 -0.076 0.036
- joint front_right_wheel_joint: limit effort=10 velocity=10 -> lower=-1.5708 upper=1.5708 effort=1 velocity=10
- joint rear_left_wheel_joint: limit effort=10 velocity=10 -> lower=-1.5708 upper=1.5708  effort=1 velocity=10; origin xyz=-0.095 0.076 0.0375 -> xyz=-0.1025 0.076 0.036
- joint rear_right_wheel_joint: limit effort=10 velocity=10 -> lower=-1.5708 upper=1.5708  effort=1 velocity=10; origin xyz=-0.095 -0.076 0.0375 -> xyz=-0.1025 -0.076 0.036

File: src/ackermann_robot/urdf/ackermann_robot.xacro (robot description, xacro)
@@ -7,12 +7,12 @@
   <xacro:property name="chassis_length" value="0.27"/>
   <xacro:property name="chassis_width"  value="0.1205"/>
-  <xacro:property name="chassis_height" value="0.002"/>
-  <xacro:property name="chassis_mass"   value="0.126"/>
+  <xacro:property name="chassis_height" value="0.00"/>
+  <xacro:property name="chassis_mass"   value="0.13442"/>
   <!-- Wheels -->
-  <xacro:property name="wheel_radius" value="0.0375"/>
+  <xacro:property name="wheel_radius" value="0.036"/>
   <xacro:property name="wheel_width"  value="0.03"/>
-  <xacro:property name="wheel_mass"   value="0.05"/>
+  <xacro:property name="wheel_mass"   value="0.0677"/>
   <!-- Geometry -->
-  <xacro:property name="wheelbase" value="0.19"/>
+  <xacro:property name="wheelbase" value="0.205"/>
   <xacro:property name="track" value="0.152"/>
   <!-- Dual plate chassis -->
@@ -24,5 +24,5 @@
   <xacro:property name="standoff_y" value="${chassis_width/2 - 0.02}"/>
   <!-- Materials -->
-  <material name="chassis_black">
+  <material name="chassis_red">
     <color rgba="1.0 0.0 0.0 1"/>
   </material>
@@ -40,28 +40,26 @@
   <link name="chassis_link">
     <inertial>
-      <origin xyz="0 0 0"/>
+      <origin xyz="0 0 ${chassis_height/2}"/>
       <mass value="${chassis_mass}"/>
       <inertia
-        ixx="0.002" ixy="0" ixz="0"
-        iyy="0.002" iyz="0"
-        izz="0.002"/>
-    </inertial>
+        ixx="1.50903123e-04" ixy="4.70052075e-08" ixz="6.59784866e-15"
+        iyy="8.14177826e-04" iyz="1.01460270e-15"
+        izz="9.64991335e-04"/>
+      </inertial>
     <!-- Bottom plate -->
     <visual>
-      <origin xyz="${-chassis_length/100} ${-chassis_width/100} ${wheel_radius + plate_thickness/2}" rpy="0 0 1.5708"/>
-      <geometry>
-        <mesh filename="/home/mohana/robot_ws/install/ackermann_robot/share/ackermann_robot/meshes/chassis_visual.stl"
-        scale="0.001 0.001 0.001"/>
-      </geometry>
-      <material name="chassis_black"/>
+      <origin xyz="0 0 ${wheel_radius + plate_thickness/2}" rpy="0 0 0"/>
+      <geometry>
+        <mesh filename="/home/mohana/robot_ws/src/ackermann_robot/meshes/chassis_visual.stl" scale="0.001 0.001 0.001"/>
+      </geometry>
+      <material name="chassis_red"/>
     </visual>
     <!-- Top plate -->
     <visual>
-      <origin xyz="${-chassis_length/100} ${-chassis_width/100} ${wheel_radius + plate_thickness + standoff_height + plate_thickness/2}" rpy="0 0 1.5708"/>
-      <geometry>
-        <mesh filename="/home/mohana/robot_ws/install/ackermann_robot/share/ackermann_robot/meshes/chassis_visual.stl"
-        scale="0.001 0.001 0.001"/>
-      </geometry>
-      <material name="chassis_black"/>
+      <origin xyz="0 0 ${wheel_radius + plate_thickness/2 + plate_thickness + standoff_height}" rpy="0 0 0"/>
+      <geometry>
+        <mesh filename="/home/mohana/robot_ws/src/ackermann_robot/meshes/chassis_visual.stl" scale="0.001 0.001 0.001"></mesh>
+      </geometry>
+      <material name="chassis_red"/>
     </visual>
     <!-- Front left standoff -->
@@ -120,12 +118,12 @@
         <mass value="${wheel_mass}"/>
         <inertia
-          ixx="3e-5" ixy="0" ixz="0"
-          iyy="3e-5" iyz="0"
-          izz="3e-5"/>
+          ixx="3.21561728e-05" ixy="1.40375656e-15" ixz="-3.63476706e-15"
+          iyy="5.65938896e-05" iyz="-1.35718707e-16"
+          izz="3.21561633e-05"/>
       </inertial>
       <visual>
-        <origin rpy="1.5708 0 0"/>
-        <geometry>
-          <mesh filename="/home/mohana/robot_ws/install/ackermann_robot/share/ackermann_robot/meshes/wheel_visual.stl"
+        <origin rpy=" 0 0 3.1412"/>
+        <geometry>
+          <mesh filename="/home/mohana/robot_ws/src/ackermann_robot/meshes/${name}_wheel.stl"
           scale="0.001 0.001 0.001"/>
         </geometry>
@@ -137,33 +135,16 @@
           <cylinder radius="${wheel_radius}" length="${wheel_width}"/>
         </geometry>
-          <surface>
-            <friction>
-              <ode>
-                <mu>0.5</mu>
-                <mu2>1.0</mu2>
-                <fdir1>0 0 1</fdir1>
-              </ode>
-              <bullet>
-                <friction>0.5</friction>
-                <friction2>1</friction2>
-                <rolling_friction>0.1</rolling_friction>
-              </bullet>
-            </friction>
-          </surface>
       </collision>
     </link>
     <!-- Gazebo friction for wheels -->
-    <gazebo reference="${name}_wheel_link">
+    <!-- <gazebo reference="${name}_wheel_link">
       <mu1>0.8</mu1>
       <mu2>0.8</mu2>
-      <kp>1000000.0</kp>
-      <kd>100.0</kd>
-    </gazebo>
-    <joint name="${name}_wheel_joint" type="revolute">
+    </gazebo> -->
+    <joint name="${name}_wheel_joint" type="continuous">
       <parent link="chassis_link"/>
       <child link="${name}_wheel_link"/>
       <origin xyz="${x} ${y} ${wheel_radius}"/>
       <axis xyz="0 1 0"/>
-      <limit effort="10" velocity="10"/>
     </joint>
   </xacro:macro>
@@ -188,5 +169,5 @@
       <origin xyz="${x} ${y} ${wheel_radius}"/>
       <axis xyz="0 0 1"/>
-      <limit lower="-0.6" upper="0.6" effort="25" velocity="2"/>
+      <limit lower="-0.6" upper="0.6" effort="10" velocity="2"/>
     </joint>
     <!-- wheel -->
@@ -200,8 +181,8 @@
       </inertial>
       <visual>
-        <origin rpy="1.5708 0 0"/>
+        <origin rpy="0 0 3.1412"/>
         <geometry>
           <!-- <cylinder radius="${wheel_radius}" length="${wheel_width}"/> -->
-        <mesh filename="/home/mohana/robot_ws/install/ackermann_robot/share/ackermann_robot/meshes/wheel_visual.stl"
+        <mesh filename="/home/mohana/robot_ws/src/ackermann_robot/meshes/${name}_wheel.stl"
         scale="0.001 0.001 0.001"/>
         </geometry>
@@ -213,32 +194,15 @@
           <cylinder radius="${wheel_radius}" length="${wheel_width}"/>
         </geometry>
-          <surface>
-            <friction>
-              <ode>
-                <mu>0.5</mu>
-                <mu2>1.0</mu2>
-                <fdir1>0 0 1</fdir1>
-              </ode>
-              <bullet>
-                <friction>0.5</friction>
-                <friction2>1</friction2>
-                <rolling_friction>0.1</rolling_friction>
-              </bullet>
-            </friction>
-          </surface>
       </collision>
     </link>
     <!-- Gazebo friction for wheels -->
-    <gazebo reference="${name}_wheel_link">
-      <mu1>0.8</mu1>
+    <!-- <gazebo reference="${name}_wheel_link">
+      <mu1>1.0</mu1>
       <mu2>0.8</mu2>
-      <kp>1000000.0</kp>
-      <kd>100.0</kd>
-    </gazebo>
-    <joint name="${name}_wheel_joint" type="revolute">
+    </gazebo> -->
+    <joint name="${name}_wheel_joint" type="continuous">
       <parent link="${name}_steer_link"/>
       <child link="${name}_wheel_link"/>
       <axis xyz="0 1 0"/>
-      <limit effort="10" velocity="10"/>
     </joint>
   </xacro:macro>
@@ -269,8 +233,6 @@
   <!-- Physics properties for chassis -->
   <!-- <gazebo reference="chassis_link">
-    <mu1>0.2</mu1>
-    <mu2>0.2</mu2>
-    <kp>1000000.0</kp>
-    <kd>100.0</kd>
+    <mu1>0.8</mu1>
+    <mu2>0.8</mu2>
   </gazebo> -->
   <gazebo>
@@ -289,6 +251,4 @@
       <wheel_radius>${wheel_radius}</wheel_radius>
       <steering_limit>0.5</steering_limit>
-      <!-- <max_velocity>1.0</max_velocity>
-      <max_acceleration>2.0</max_acceleration> -->
       <topic>/cmd_vel</topic>
       <odom_topic>/odometry</odom_topic>
@@ -301,5 +261,4 @@
       filename="gz-sim-joint-state-publisher-system"
       name="gz::sim::systems::JointStatePublisher"/>
-      <frame_id>base_link</frame_id>
   </gazebo>
 </robot>
