Commit message: "add all ros2 works"

File: src/ackermann_robot/urdf/ackermann_robot.urdf (robot description, URDF)
Before this commit: robot ackermann_robot, 8 links, 7 joints
Links:
- link chassis_link: geometry collision box size=0.27 0.1205 0.0; visual cylinder length=0.04 radius=0.004
Joints:
- joint front_left_steer_joint: limit lower=-0.6 upper=0.6 effort=1 velocity=2 -> lower=-0.6 upper=0.6 effort=10 velocity=2
- joint front_left_wheel_joint: limit lower=-1.5708 upper=1.5708 effort=1 velocity=10 -> (none); type revolute -> continuous
- joint front_right_steer_joint: limit lower=-0.6 upper=0.6 effort=1 velocity=2 -> lower=-0.6 upper=0.6 effort=10 velocity=2
- joint front_right_wheel_joint: limit lower=-1.5708 upper=1.5708 effort=1 velocity=10 -> (none); type revolute -> continuous
- joint rear_left_wheel_joint: limit lower=-1.5708 upper=1.5708  effort=1 velocity=10 -> (none); type revolute -> continuous
- joint rear_right_wheel_joint: limit lower=-1.5708 upper=1.5708  effort=1 velocity=10 -> (none); type revolute -> continuous

File: src/ackermann_robot/urdf/ackermann_robot.xacro (robot description, xacro)
@@ -4,8 +4,12 @@
   <!-- Real hardware values  -->
   <!-- ===================== -->
+  <!-- Dual plate chassis -->
+  <xacro:property name="plate_thickness" value="0.002"/>
+  <xacro:property name="standoff_height" value="0.04"/>
+  <xacro:property name="standoff_radius" value="0.004"/>
   <!-- Chassis -->
   <xacro:property name="chassis_length" value="0.27"/>
   <xacro:property name="chassis_width"  value="0.1205"/>
-  <xacro:property name="chassis_height" value="0.00"/>
+  <xacro:property name="chassis_height" value="${2*plate_thickness + standoff_height}"/>
   <xacro:property name="chassis_mass"   value="0.13442"/>
   <!-- Wheels -->
@@ -16,8 +20,4 @@
   <xacro:property name="wheelbase" value="0.205"/>
   <xacro:property name="track" value="0.152"/>
-  <!-- Dual plate chassis -->
-  <xacro:property name="plate_thickness" value="0.002"/>
-  <xacro:property name="standoff_height" value="0.04"/>
-  <xacro:property name="standoff_radius" value="0.004"/>
   <!-- Standoff positions -->
   <xacro:property name="standoff_x" value="${chassis_length/2 - 0.02}"/>
@@ -97,5 +97,5 @@
     <!-- Collision: simple box for stable physics -->
     <collision>
-      <origin xyz="0 0 ${chassis_height/2}"/>
+      <origin xyz="0 0 ${wheel_radius + chassis_height/2}"/>
       <geometry>
         <box size="${chassis_length} ${chassis_width} ${chassis_height}"/>
@@ -107,5 +107,5 @@
     <parent link="base_link"/>
     <child link="chassis_link"/>
-    <origin xyz="0 0 ${wheel_radius}" rpy="0 0 0"/>
+    <origin xyz="0 0 0" rpy="0 0 0"/>
   </joint>
   <!-- ===================== -->
@@ -138,8 +138,8 @@
     </link>
     <!-- Gazebo friction for wheels -->
-    <!-- <gazebo reference="${name}_wheel_link">
-      <mu1>0.8</mu1>
-      <mu2>0.8</mu2>
-    </gazebo> -->
+    <gazebo reference="${name}_wheel_link">
+      <mu1>1.0</mu1>
+      <mu2>1.0</mu2>
+    </gazebo>
     <joint name="${name}_wheel_joint" type="continuous">
       <parent link="chassis_link"/>
@@ -197,8 +197,8 @@
     </link>
     <!-- Gazebo friction for wheels -->
-    <!-- <gazebo reference="${name}_wheel_link">
+    <gazebo reference="${name}_wheel_link">
       <mu1>1.0</mu1>
-      <mu2>0.8</mu2>
-    </gazebo> -->
+      <mu2>1.0</mu2>
+    </gazebo>
     <joint name="${name}_wheel_joint" type="continuous">
       <parent link="${name}_steer_link"/>
@@ -232,8 +232,8 @@
   <!-- ===================== -->
   <!-- Physics properties for chassis -->
-  <!-- <gazebo reference="chassis_link">
+  <gazebo reference="chassis_link">
     <mu1>0.8</mu1>
     <mu2>0.8</mu2>
-  </gazebo> -->
+  </gazebo>
   <gazebo>
     <plugin

Commit message: MG400 full setup

File: src/ackermann_robot/urdf/ackermann_robot.urdf (robot description, URDF)
Before this commit: robot ackermann_robot, 8 links, 7 joints
Links:
- added link front_camera_link; visual box size=0.02 0.02 0.02
- added link imu_link, mass 0.001
- added link left_camera_link; visual box size=0.02 0.02 0.02
- added link rear_camera_link; visual box size=0.02 0.02 0.02
- added link right_camera_link; visual box size=0.02 0.02 0.02
- link chassis_link: geometry collision box size=0.27 0.1205 0.044; visual cylinder length=0.04 radius=0.004
- link front_left_wheel_link: geometry collision cylinder length=0.03 radius=0.036; visual mesh filename=package://ackermann_robot/meshes/front_left_wheel.stl scale=0.001 0.001 0.001
- link front_right_wheel_link: geometry collision cylinder length=0.03 radius=0.036; visual mesh filename=package://ackermann_robot/meshes/front_right_wheel.stl scale=0.001 0.001 0.001
- link rear_left_wheel_link: geometry collision cylinder length=0.03 radius=0.036; visual mesh filename=package://ackermann_robot/meshes/rear_left_wheel.stl scale=0.001 0.001 0.001
- link rear_right_wheel_link: geometry collision cylinder length=0.03 radius=0.036; visual mesh filename=package://ackermann_robot/meshes/rear_right_wheel.stl scale=0.001 0.001 0.001
Joints:
- added joint front_camera_joint: type fixed, parent base_link, child front_camera_link, origin xyz=0.135 0.0 0.08 rpy=0.0 0.0 0.0
- added joint imu_joint: type fixed, parent base_link, child imu_link, origin xyz=0 0 0.05 rpy=0 0 0
- added joint left_camera_joint: type fixed, parent base_link, child left_camera_link, origin xyz=0.0 0.06025 0.08 rpy=0.0 0.0 1.5708
- added joint rear_camera_joint: type fixed, parent base_link, child rear_camera_link, origin xyz=-0.135 0.0 0.08 rpy=0.0 0.0 3.14159
- added joint right_camera_joint: type fixed, parent base_link, child right_camera_link, origin xyz=0.0 -0.06025 0.08 rpy=0.0 0.0 -1.5708
- joint base_to_chassis: origin xyz=0 0 0.036 rpy=0 0 0 -> xyz=0 0 0 rpy=0 0 0

File: src/ackermann_robot/urdf/ackermann_robot.xacro (robot description, xacro)
@@ -1,4 +1,5 @@
 <?xml version="1.0"?>
 <robot name="ackermann_robot" xmlns:xacro="http://www.ros.org/wiki/xacro">
+  <xacro:include filename="$(find ackermann_robot)/urdf/all_sensors.xacro" />
   <!-- ===================== -->
   <!-- Real hardware values  -->
@@ -11,5 +12,5 @@
   <xacro:property name="chassis_length" value="0.27"/>
   <xacro:property name="chassis_width"  value="0.1205"/>
-  <xacro:property name="chassis_height" value="${2*plate_thickness + standoff_height}"/>
+  <xacro:property name="chassis_height" value="${3*plate_thickness + 2*standoff_height}"/>
   <xacro:property name="chassis_mass"   value="0.13442"/>
   <!-- Wheels -->
@@ -51,13 +52,21 @@
       <origin xyz="0 0 ${wheel_radius + plate_thickness/2}" rpy="0 0 0"/>
       <geometry>
-        <mesh filename="/home/mohana/robot_ws/src/ackermann_robot/meshes/chassis_visual.stl" scale="0.001 0.001 0.001"/>
+        <mesh filename="package://ackermann_robot/meshes/chassis_visual.stl" scale="0.001 0.001 0.001"/>
       </geometry>
       <material name="chassis_red"/>
     </visual>
+    <!-- Middle plate -->
+    <visual>
+      <origin xyz="0 0 ${wheel_radius + plate_thickness/2 + plate_thickness + standoff_height}" rpy="0 0 0"/>
+      <geometry>
+        <mesh filename="package://ackermann_robot/meshes/chassis_visual.stl" scale="0.001 0.001 0.001"></mesh>
+      </geometry>
+      <material name="chassis_red"/>
+    </visual>
     <!-- Top plate -->
     <visual>
-      <origin xyz="0 0 ${wheel_radius + plate_thickness/2 + plate_thickness + standoff_height}" rpy="0 0 0"/>
-      <geometry>
-        <mesh filename="/home/mohana/robot_ws/src/ackermann_robot/meshes/chassis_visual.stl" scale="0.001 0.001 0.001"></mesh>
+      <origin xyz="0 0 ${wheel_radius + plate_thickness/2 + 2*plate_thickness + 2*standoff_height}" rpy="0 0 0"/>
+      <geometry>
+        <mesh filename="package://ackermann_robot/meshes/chassis_visual.stl" scale="0.001 0.001 0.001"></mesh>
       </geometry>
       <material name="chassis_red"/>
@@ -90,4 +99,36 @@
     <visual>
       <origin xyz="-${standoff_x} -${standoff_y} ${wheel_radius + plate_thickness + standoff_height/2}" rpy="0 0 0"/>
+      <geometry>
+        <cylinder radius="${standoff_radius}" length="${standoff_height}"/>
+      </geometry>
+      <material name="wheel_black"/>
+    </visual>
+    <!-- Upper Front left standoff -->
+    <visual>
+      <origin xyz="${standoff_x} ${standoff_y} ${wheel_radius + 2*plate_thickness + standoff_height + standoff_height/2}" rpy="0 0 0"/>
+      <geometry>
+        <cylinder radius="${standoff_radius}" length="${standoff_height}"/>
+      </geometry>
+      <material name="wheel_black"/>
+    </visual>
+    <!-- Upper Front right -->
+    <visual>
+      <origin xyz="${standoff_x} -${standoff_y} ${wheel_radius + 2*plate_thickness + standoff_height + standoff_height/2}" rpy="0 0 0"/>
+      <geometry>
+        <cylinder radius="${standoff_radius}" length="${standoff_height}"/>
+      </geometry>
+      <material name="wheel_black"/>
+    </visual>
+    <!-- Upper Rear left -->
+    <visual>
+      <origin xyz="-${standoff_x} ${standoff_y} ${wheel_radius + 2*plate_thickness + standoff_height + standoff_height/2}" rpy="0 0 0"/>
+      <geometry>
+        <cylinder radius="${standoff_radius}" length="${standoff_height}"/>
+      </geometry>
+      <material name="wheel_black"/>
+    </visual>
+    <!-- Upper Rear right -->
+    <visual>
+      <origin xyz="-${standoff_x} -${standoff_y} ${wheel_radius + 2*plate_thickness + standoff_height + standoff_height/2}" rpy="0 0 0"/>
       <geometry>
         <cylinder radius="${standoff_radius}" length="${standoff_height}"/>
@@ -125,5 +166,5 @@
         <origin rpy=" 0 0 3.1412"/>
         <geometry>
-          <mesh filename="/home/mohana/robot_ws/src/ackermann_robot/meshes/${name}_wheel.stl"
+          <mesh filename="package://ackermann_robot/meshes/${name}_wheel.stl"
           scale="0.001 0.001 0.001"/>
         </geometry>
@@ -184,5 +225,5 @@
         <geometry>
           <!-- <cylinder radius="${wheel_radius}" length="${wheel_width}"/> -->
-        <mesh filename="/home/mohana/robot_ws/src/ackermann_robot/meshes/${name}_wheel.stl"
+        <mesh filename="package://ackermann_robot/meshes/${name}_wheel.stl"
         scale="0.001 0.001 0.001"/>
         </geometry>
@@ -237,28 +278,33 @@
   </gazebo>
   <gazebo>
-    <plugin
-      filename="gz-sim-ackermann-steering-system"
-      name="gz::sim::systems::AckermannSteering">
+    <plugin filename="gz-sim-ackermann-steering-system" name="gz::sim::systems::AckermannSteering">
       <left_steering_joint>front_left_steer_joint</left_steering_joint>
       <right_steering_joint>front_right_steer_joint</right_steering_joint>
-      <left_joint>front_left_wheel_joint</left_joint>
       <left_joint>rear_left_wheel_joint</left_joint>
-      <right_joint>front_right_wheel_joint</right_joint>
       <right_joint>rear_right_wheel_joint</right_joint>
-      <wheel_base>${wheelbase}</wheel_base>
-      <wheel_separation>${track}</wheel_separation>
-      <kingpin_width>${track}</kingpin_width>
-      <wheel_radius>${wheel_radius}</wheel_radius>
+      <wheel_base>0.205</wheel_base>
+      <wheel_separation>0.152</wheel_separation>
+      <kingpin_width>0.152</kingpin_width>
+      <wheel_radius>0.036</wheel_radius>
       <steering_limit>0.5</steering_limit>
       <topic>/cmd_vel</topic>
-      <odom_topic>/odometry</odom_topic>
-      <tf_topic>/tf</tf_topic>
+      <odom_topic>/odom</odom_topic>
+      <frame_id>odom</frame_id>
+      <child_frame_id>base_link</child_frame_id>
       <odom_publish_frequency>30</odom_publish_frequency>
     </plugin>
-  </gazebo>
-  <gazebo>
-    <plugin
-      filename="gz-sim-joint-state-publisher-system"
-      name="gz::sim::systems::JointStatePublisher"/>
+    <plugin filename="gz-sim-pose-publisher-system" name="gz::sim::systems::PosePublisher">
+      <publish_link_pose>true</publish_link_pose>
+      <publish_sensor_pose>true</publish_sensor_pose>
+      <publish_model_pose>true</publish_model_pose>
+      <use_pose_vector_msg>true</use_pose_vector_msg>
+    </plugin>
+    <plugin filename="gz-sim-odometry-publisher-system" name="gz::sim::systems::OdometryPublisher">
+      <odom_frame>ground_truth_odom</odom_frame>
+      <robot_base_frame>base_link</robot_base_frame>
+      <odom_topic>/ground_truth_odom</odom_topic>
+      <dimensions>3</dimensions>
+    </plugin>
+    <plugin filename="gz-sim-joint-state-publisher-system" name="gz::sim::systems::JointStatePublisher"/>
   </gazebo>
 </robot>
