Commit message: latests acker and added Qualcomm Robotics Sim

File: src/ackermann_robot/urdf/ackermann_robot.xacro (robot description, xacro)
@@ -2,23 +2,4 @@
 <robot name="ackermann_robot" xmlns:xacro="http://www.ros.org/wiki/xacro">
   <xacro:include filename="$(find ackermann_robot)/urdf/all_sensors.xacro" />
-  <!-- ===================== -->
-  <!-- Real hardware values  -->
-  <!-- ===================== -->
-  <!-- Dual plate chassis -->
-  <xacro:property name="plate_thickness" value="0.002"/>
-  <xacro:property name="standoff_height" value="0.04"/>
-  <xacro:property name="standoff_radius" value="0.004"/>
-  <!-- Chassis -->
-  <xacro:property name="chassis_length" value="0.27"/>
-  <xacro:property name="chassis_width"  value="0.1205"/>
-  <xacro:property name="chassis_height" value="${3*plate_thickness + 2*standoff_height}"/>
-  <xacro:property name="chassis_mass"   value="0.13442"/>
-  <!-- Wheels -->
-  <xacro:property name="wheel_radius" value="0.036"/>
-  <xacro:property name="wheel_width"  value="0.03"/>
-  <xacro:property name="wheel_mass"   value="0.0677"/>
-  <!-- Geometry -->
-  <xacro:property name="wheelbase" value="0.205"/>
-  <xacro:property name="track" value="0.152"/>
   <!-- Standoff positions -->
   <xacro:property name="standoff_x" value="${chassis_length/2 - 0.02}"/>
@@ -36,4 +17,10 @@
   <!-- Robot center reference -->
   <link name="base_link"/>
+  <link name="base_footprint"></link>
+  <joint name="base_footprint_joint" type="fixed">
+      <parent link="base_link"/>
+      <child link="base_footprint"/>
+      <origin xyz="0 0 0" rpy="0 0 0"/>
+  </joint>
   <!-- ===================== -->
   <!-- Chassis               -->
@@ -148,5 +135,5 @@
     <parent link="base_link"/>
     <child link="chassis_link"/>
-    <origin xyz="0 0 0" rpy="0 0 0"/>
+    <origin xyz="${wheelbase/2} 0 0" rpy="0 0 0"/>
   </joint>
   <!-- ===================== -->
@@ -287,5 +274,5 @@
       <kingpin_width>0.152</kingpin_width>
       <wheel_radius>0.036</wheel_radius>
-      <steering_limit>0.5</steering_limit>
+      <steering_limit>1.0</steering_limit>
       <topic>/cmd_vel</topic>
       <odom_topic>/odom</odom_topic>
@@ -294,5 +281,5 @@
       <odom_publish_frequency>30</odom_publish_frequency>
     </plugin>
-    <plugin filename="gz-sim-pose-publisher-system" name="gz::sim::systems::PosePublisher">
+    <!-- <plugin filename="gz-sim-pose-publisher-system" name="gz::sim::systems::PosePublisher">
       <publish_link_pose>true</publish_link_pose>
       <publish_sensor_pose>true</publish_sensor_pose>
@@ -305,6 +292,88 @@
       <odom_topic>/ground_truth_odom</odom_topic>
       <dimensions>3</dimensions>
+    </plugin> -->
+    <plugin filename="gz-sim-joint-state-publisher-system" name="gz::sim::systems::JointStatePublisher">
+      <topic>/joint_states</topic>
     </plugin>
-    <plugin filename="gz-sim-joint-state-publisher-system" name="gz::sim::systems::JointStatePublisher"/>
   </gazebo>
+  <material name="arduino_blue">
+    <color rgba="0.1 0.5 0.5 1"/>
+  </material>
+  <material name="sbc_green">
+    <color rgba="0.1 0.6 0.1 1"/>
+  </material>
+  <!-- ===================== -->
+  <!-- Extra Visuals         -->
+  <!-- ===================== -->
+  <!-- Front steering servo -->
+  <link name="front_servo_link">
+    <visual>
+      <geometry>
+        <box size="0.03 0.05 0.03"/>
+      </geometry>
+      <material name="wheel_black"/>
+    </visual>
+  </link>
+  <joint name="front_servo_joint" type="fixed">
+    <parent link="chassis_link"/>
+    <child link="front_servo_link"/>
+    <origin rpy="0 0 0" xyz="0.1 0 ${wheel_radius*1.5}"/>
+  </joint>
+  <!-- Rear wheel motors -->
+  <link name="rear_left_motor_link">
+    <visual>
+      <origin rpy="1.5708 0 0"/>
+      <geometry>
+        <cylinder length="0.03" radius="0.02"/>
+      </geometry>
+      <material name="wheel_black"/>
+    </visual>
+  </link>
+  <joint name="rear_left_motor_joint" type="fixed">
+    <parent link="chassis_link"/>
+    <child link="rear_left_motor_link"/>
+    <origin rpy="0 0 0" xyz="-0.1025 0.05 0.036"/>
+  </joint>
+  <link name="rear_right_motor_link">
+    <visual>
+      <origin rpy="1.5708 0 0"/>
+      <geometry>
+        <cylinder length="0.03" radius="0.02"/>
+      </geometry>
+      <material name="wheel_black"/>
+    </visual>
+  </link>
+  <joint name="rear_right_motor_joint" type="fixed">
+    <parent link="chassis_link"/>
+    <child link="rear_right_motor_link"/>
+    <origin rpy="0 0 0" xyz="-0.1025 -0.05 0.036"/>
+  </joint>
+  <!-- Arduino -->
+  <link name="arduino_link">
+    <visual>
+      <geometry>
+        <box size="0.075 0.053 0.01"/>
+      </geometry>
+      <material name="arduino_blue"/>
+    </visual>
+  </link>
+  <joint name="arduino_joint" type="fixed">
+    <parent link="chassis_link"/>
+    <child link="arduino_link"/>
+    <origin rpy="0 0 0" xyz="-${wheelbase/4} 0.0 0.045"/>
+  </joint>
+  <!-- SBC -->
+  <link name="sbc_link">
+    <visual>
+      <geometry>
+        <box size="0.085 0.056 0.015"/>
+      </geometry>
+      <material name="sbc_green"/>
+    </visual>
+  </link>
+  <joint name="sbc_joint" type="fixed">
+    <parent link="chassis_link"/>
+    <child link="sbc_link"/>
+    <origin rpy="0 0 0" xyz="-${wheelbase/4} 0.0 0.085"/>
+  </joint>
 </robot>

File: src/ackermann_robot/urdf/all_sensors.xacro (robot description, xacro)
@@ -1,13 +1,40 @@
 <?xml version="1.0" ?>
 <robot xmlns:xacro="http://www.ros.org/wiki/xacro">
+  <!-- ===================== -->
+  <!-- Real hardware values  -->
+  <!-- ===================== -->
+  <!-- Dual plate chassis -->
+  <xacro:property name="plate_thickness" value="0.002"/>
+  <xacro:property name="standoff_height" value="0.04"/>
+  <xacro:property name="standoff_radius" value="0.004"/>
+  <!-- Chassis -->
+  <xacro:property name="chassis_length" value="0.27"/>
+  <xacro:property name="chassis_width"  value="0.1205"/>
+  <xacro:property name="chassis_height" value="${3*plate_thickness + 2*standoff_height}"/>
+  <xacro:property name="chassis_mass"   value="0.13442"/>
+  <!-- Wheels -->
+  <xacro:property name="wheel_radius" value="0.036"/>
+  <xacro:property name="wheel_width"  value="0.03"/>
+  <xacro:property name="wheel_mass"   value="0.0677"/>
+  <!-- Geometry -->
+  <xacro:property name="wheelbase" value="0.21"/>
+  <xacro:property name="track" value="0.152"/>
+  <xacro:property name="imu_z" value="0.05"/>
+  <xacro:property name="lidar_z" value="0.14"/>
+  <xacro:property name="lidar_x_offset" value="0.05"/>
+  <xacro:property name="camera_size" value="0.02" />
+  <xacro:property name="camera_z" value="${wheel_radius + chassis_height}"/>
+  <xacro:property name="cam_pitch" value="0.3490"/>
   <xacro:include filename="$(find ackermann_robot)/urdf/sensors_cameras.xacro" />
   <xacro:include filename="$(find ackermann_robot)/urdf/sensors_imu.xacro" />
+  <xacro:include filename="$(find ackermann_robot)/urdf/sensors_lidar.xacro" />
   <xacro:sensor_imu name="imu" parent="base_link">
-    <origin xyz="0 0 0.05" rpy="0 0 0"/>
+    <origin x="${wheelbase/2}" y="0" z="${imu_z}" rpy="0 0 0"/>
   </xacro:sensor_imu>
+  <xacro:sensor_lidar name="lidar" x="${wheelbase/2 + lidar_x_offset}" y="0.0" z="${lidar_z}" roll="0.0" pitch="0.0" yaw="0.0"/>
   <xacro:wide_angle_camera
     name="front"
-    x="0.135" y="0.0" z="0.08"
-    roll="0.0" pitch="0.0" yaw="0.0"
+    x="${wheelbase/2 + chassis_length/2}" y="0.0" z="${camera_z}"
+    roll="0.0" pitch="${cam_pitch}" yaw="0.0"
     width="1280" height="720" fov="2.0944"
     fx="369.5" fy="369.5" cx="640" cy="360"
@@ -15,6 +42,6 @@
   <xacro:wide_angle_camera
     name="left"
-    x="0.0" y="0.06025" z="0.08"
-    roll="0.0" pitch="0.0" yaw="1.5708"
+    x="${wheelbase/2}" y="${chassis_width/2}" z="${camera_z}"
+    roll="0.0" pitch="${cam_pitch}" yaw="1.5708"
     width="1280" height="720" fov="2.0944"
     fx="369.5" fy="369.5" cx="640" cy="360"
@@ -22,6 +49,6 @@
   <xacro:wide_angle_camera
     name="right"
-    x="0.0" y="-0.06025" z="0.08"
-    roll="0.0" pitch="0.0" yaw="-1.5708"
+    x="${wheelbase/2}" y="-${chassis_width/2}" z="${camera_z}"
+    roll="0.0" pitch="${cam_pitch}" yaw="-1.5708"
     width="1280" height="720" fov="2.0944"
     fx="369.5" fy="369.5" cx="640" cy="360"
@@ -29,6 +56,6 @@
   <xacro:wide_angle_camera
     name="rear"
-    x="-0.135" y="0.0" z="0.08"
-    roll="0.0" pitch="0.0" yaw="3.14159"
+    x="${wheelbase/2 - chassis_length/2}" y="0.0" z="${camera_z}"
+    roll="0.0" pitch="${cam_pitch}" yaw="3.14159"
     width="1280" height="720" fov="2.0944"
     fx="369.5" fy="369.5" cx="640" cy="360"

File: src/ackermann_robot/urdf/sensors_lidar.xacro (robot description, xacro)
@@ -1,24 +1,24 @@
 <?xml version="1.0" ?>
 <robot xmlns:xacro="http://www.ros.org/wiki/xacro">
-<!-- Macro for Lidar (Sonar/Laser) -->
-  <xacro:macro name="sensor_lidar" params="name parent *origin update_rate:=5 samples:=1 resolution:=1 min_angle:=0 max_angle:=0 range_min:=0.2 range_max:=5 visualize:=0">
+<!-- Macro for GPU Lidar -->
+  <xacro:macro name="sensor_lidar" params="name x y z roll pitch yaw update_rate:=10 samples:=360 resolution:=1 min_angle:=0.0 max_angle:=6.28318 range_min:=0.1 range_max:=5.0">
     <link name="${name}_link">
       <visual>
         <geometry>
-          <cylinder radius="0.01" length="0.01"/>
+          <cylinder radius="0.03" length="0.05"/>
         </geometry>
-        <material name="yellow">
-            <color rgba="1 1 0 1"/>
+        <material name="blue">
+            <color rgba="0 0 1 1"/>
         </material>
-        </visual>
+      </visual>
       <inertial>
-        <mass value="0.01"/>
-        <inertia ixx="1e-5" ixy="0" ixz="0" iyy="1e-5" iyz="0" izz="1e-5"/>
+        <mass value="0.1"/>
+        <inertia ixx="1e-4" ixy="0" ixz="0" iyy="1e-4" iyz="0" izz="1e-4"/>
       </inertial>
     </link>
     <joint name="${name}_joint" type="fixed">
-      <parent link="${parent}"/>
+      <parent link="base_link"/>
       <child link="${name}_link"/>
-      <xacro:insert_block name="origin"/>
+      <origin xyz="${x} ${y} ${z}" rpy="${roll} ${pitch} ${yaw}" />
     </joint>
     <gazebo reference="${name}_joint">
@@ -27,5 +27,4 @@
     <gazebo reference="${name}_link">
       <sensor name="${name}_sensor" type="gpu_lidar">
-        <topic>/${name}/scan</topic>
         <lidar>
           <scan>
@@ -38,4 +37,5 @@
             <vertical>
               <samples>1</samples>
+              <resolution>1</resolution>
               <min_angle>0</min_angle>
               <max_angle>0</max_angle>
@@ -49,6 +49,8 @@
         </lidar>
         <always_on>1</always_on>
+        <visualize>true</visualize>
+        <topic>/scan</topic>
+        <gz_frame_id>${name}_link</gz_frame_id>
         <update_rate>${update_rate}</update_rate>
-        <visualize>${visualize}</visualize>
       </sensor>
     </gazebo>

Commit message: "rtabmap integration"

File: src/ackermann_robot/urdf/ackermann_robot.xacro (robot description, xacro)
@@ -16,10 +16,17 @@
   <!-- ===================== -->
   <!-- Robot center reference -->
-  <link name="base_link"/>
+  <!-- <link name="base_link"/>
   <link name="base_footprint"></link>
   <joint name="base_footprint_joint" type="fixed">
       <parent link="base_link"/>
       <child link="base_footprint"/>
-      <origin xyz="0 0 0" rpy="0 0 0"/>
+      <origin xyz="0 0 ${wheel_radius}" rpy="0 0 0"/>
+  </joint> -->
+  <link name="base_link"></link>
+  <link name="base_footprint"></link>
+  <joint name="base_footprint_joint" type="fixed">
+      <parent link="base_link"/>
+      <child link="base_footprint"/>
+      <origin xyz="0 0 -${chassis_height/2}" rpy="0 0 0"/>
   </joint>
   <!-- ===================== -->

File: src/ackermann_robot/urdf/all_sensors.xacro (robot description, xacro)
@@ -61,3 +61,9 @@
     fx="369.5" fy="369.5" cx="640" cy="360"
     k1="0.0" k2="0.0" k3="0.0" p1="0.0" p2="0.0" />
+  <xacro:rgbd_camera
+    name="depth"
+    x="${wheelbase}" y="0.0" z="${camera_z/1.3}"
+    roll="0.0" pitch="0.0" yaw="0.0"
+    width="1280" height="720" fov="2.0944"
+    k1="0.0" k2="0.0" k3="0.0" p1="0.0" p2="0.0" />
 </robot>

File: src/ackermann_robot/urdf/sensors_cameras.xacro (robot description, xacro)
@@ -46,18 +46,19 @@
           <!-- Lens configuration for wide angle/fisheye simulation -->
           <lens>
+            <type>equidistant</type>
             <!-- type element is mandatory -->
-            <type>custom</type>
+            <!-- <type>custom</type> -->
             <!-- manually defined mapping function r = c1*f*fun(theta/c2 + c3) -->
             <!-- More information here: https://en.wikipedia.org/wiki/Fisheye_lens#Mapping_function -->
-            <custom_function>
-              <c1>1.05</c1>
+            <!-- <custom_function>
+              <c1>1.05</c1> -->
               <!-- linear scaling -->
-              <c2>4</c2>
+              <!-- <c2>4</c2> -->
               <!-- angle scaling -->
-              <f>1.0</f>
+              <!-- <f>1.0</f> -->
               <!-- one more scaling parameter -->
-              <fun>tan</fun>
+              <!-- <fun>tan</fun> -->
               <!-- one of sin,tan,id -->
-            </custom_function>
+            <!-- </custom_function> -->
             <!-- if it is set to `true` your horizontal FOV will ramain as defined -->
             <!-- othervise it depends on lens type and custom function, if there is one -->
@@ -89,3 +90,64 @@
     </gazebo>
   </xacro:macro>
+  <xacro:macro name="rgbd_camera" params="name x y z roll pitch yaw width height fov k1 k2 k3 p1 p2">
+    <link name="${name}_camera_link">
+      <visual>
+        <origin xyz="0 0 0" rpy="0 0 0"/>
+        <geometry>
+          <box size="0.02 0.02 0.02"/>
+        </geometry>
+        <material name="wheel_black"/>
+      </visual>
+    </link>
+    <joint name="${name}_camera_joint" type="fixed">
+      <parent link="base_link"/>
+      <child link="${name}_camera_link"/>
+      <origin xyz="${x} ${y} ${z}" rpy="${roll} ${pitch} ${yaw}"/>
+    </joint>
+    <link name="${name}_camera_optical_link"/>
+    <joint name="${name}_joint" type="fixed">
+      <parent link="${name}_camera_link"/>
+      <child link="${name}_camera_optical_link"/>
+      <origin xyz="0 0 0" rpy="-1.5708 0 -1.5708"/>
+    </joint>
+    <gazebo reference="${name}_camera_link">
+      <sensor name="${name}_camera" type="rgbd_camera">
+        <camera>
+          <horizontal_fov>${fov}</horizontal_fov>
+          <image>
+            <width>${width}</width>
+            <height>${height}</height>
+          </image>
+          <clip>
+            <near>0.1</near>
+            <far>10</far>
+          </clip>
+          <distortion>
+            <k1>${k1}</k1>
+            <k2>${k2}</k2>
+            <k3>${k3}</k3>
+            <p1>${p1}</p1>
+            <p2>${p2}</p2>
+            <center>0.5 0.5</center>
+          </distortion>
+        </camera>
+        <depth_camera>
+          <clip>
+            <near>0.1</near>
+            <far>10</far>
+          </clip>
+          <noise>
+            <type>gaussian</type>
+            <mean>0.0</mean>
+            <stddev>0.01</stddev>
+          </noise>
+        </depth_camera>
+        <always_on>1</always_on>
+        <update_rate>30</update_rate>
+        <visualize>true</visualize>
+        <topic>${name}_camera</topic>
+        <gz_frame_id>${name}_camera_optical_link</gz_frame_id>
+      </sensor>
+    </gazebo>
+  </xacro:macro>
 </robot>

File: src/ackermann_robot/urdf/sensors_imu.xacro (robot description, xacro)
@@ -22,4 +22,5 @@
         <update_rate>${update_rate}</update_rate>
         <topic>/imu</topic>
+        <gz_frame_id>${name}_link</gz_frame_id>
       </sensor>
     </gazebo>
